File: Hardware/BLCtrlToPWM.kicad_pcb (KiCad board)
At the start: 2 copper layers, 62 x 50 mm, 42 parts, among them IC1 ATMEGA2560-A, Q1 Q_NMOS_GSD, Q2 Q_NMOS_GSD, Q3 Q_NMOS_GSD, Q4 Q_NMOS_GSD, Q5 Q_NMOS_GSD, Y1 16MHz

Commit message: Finished board design for version 2
Parts:
- C1, C2: value 27p -> 22p
- Y1: footprint Crystals:Crystal_HC49-SD_SMD -> Crystals:Crystal_HC49-U_Vertical
- moved SV3 48.4 mm to (25.0, -11.5), turned to 90 degrees
- moved Q5 23.1 mm to (-18.5, 16.0), turned to 180 degrees
- moved Q4 22.9 mm to (-18.5, 12.5), turned to 180 degrees
- moved Q3 22.2 mm to (-18.5, -11.5), turned to 180 degrees
- moved Q2 22.1 mm to (-18.5, -15.0), turned to 180 degrees
- moved Q1 22.1 mm to (-18.5, -18.5), turned to 180 degrees
- moved JP2 1.51 mm to (-23.5, 9.00), turned to 0 degrees
- moved JP1 1.07 mm to (-16.0, -23.2)
- moved R4 1.00 mm to (-26.0, -18.5), turned to 0 degrees
- moved R7 1.00 mm to (-26.0, 18.5)
- moved R3 1.00 mm to (-26.0, 14.0), turned to 0 degrees
- moved R5 1.00 mm to (-26.0, -14.0), turned to 0 degrees
- moved R2 1.00 mm to (-26.0, -16.0), turned to 0 degrees
- moved R6 1.00 mm to (-26.0, 16.0), turned to 0 degrees
- moved D3 0.39 mm to (-33.0, 18.5)
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Connections:
- D1 pad 2: Net-(D1-Pad2) -> +5V
- D2 pad 2: Net-(D2-Pad2) -> +5V
- D4 pad 2: Net-(D4-Pad2) -> +5V
- D5 pad 2: Net-(D5-Pad2) -> +5V
- D6 pad 2: Net-(D6-Pad2) -> +5V
- Q1 pad 3: Net-(D4-Pad1) -> Net-(Q1-Pad3)
- Q2 pad 3: Net-(D1-Pad1) -> Net-(Q2-Pad3)
- Q3 pad 3: Net-(D5-Pad1) -> Net-(Q3-Pad3)
- Q4 pad 3: Net-(D2-Pad1) -> Net-(Q4-Pad3)
- Q5 pad 3: Net-(D6-Pad1) -> Net-(Q5-Pad3)
- R2 pad 1: +5V -> Net-(D1-Pad1)
- R2 pad 2: Net-(D1-Pad2) -> Net-(Q2-Pad3)
- R3 pad 1: +5V -> Net-(D2-Pad1)
- R3 pad 2: Net-(D2-Pad2) -> Net-(Q4-Pad3)
- R4 pad 1: +5V -> Net-(D4-Pad1)
- R4 pad 2: Net-(D4-Pad2) -> Net-(Q1-Pad3)
- R5 pad 1: +5V -> Net-(D5-Pad1)
- R5 pad 2: Net-(D5-Pad2) -> Net-(Q3-Pad3)
- R6 pad 1: +5V -> Net-(D6-Pad1)
- R6 pad 2: Net-(D6-Pad2) -> Net-(Q5-Pad3)
Routing:
- net +5V: track 113.1 -> 202.8 mm, vias 3 -> 6
- net Earth: track 341.8 -> 286.0 mm, vias 32 -> 26
- net (no net): track 39.2 -> 0.50 mm, vias 2 -> 0
- net Net-(IC1-Pad63): track 0.00 -> 27.5 mm, vias 0 -> 2
- net /GREEN_LED: track 0.00 -> 22.3 mm, vias 0 -> 2
- net Net-(JP2-Pad1): track 8.24 -> 30.5 mm
- net /TX_LED: track 0.00 -> 19.4 mm, vias 0 -> 2
- net /RX_LED: track 0.00 -> 19.2 mm, vias 0 -> 2
- net Net-(IC1-Pad64): track 0.00 -> 18.2 mm, vias 0 -> 2
- net /BLUE2_LED: track 0.00 -> 17.1 mm
- net Net-(IC1-Pad45): track 57.5 -> 40.9 mm, vias 1 -> 2
- net /BLUE1_LED: track 0.60 -> 15.6 mm
- net Net-(D6-Pad2): track 7.05 -> 0.00 mm
- net Net-(D1-Pad2): track 7.05 -> 0.00 mm
- net Net-(D5-Pad2): track 7.00 -> 0.00 mm
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
Commit message: Added a side button
Parts:
- added SW1: SW_SPST, Switches:PanasonicEVQPU_SPST_NO, F.Cu at (7.00, 25.0)
Connections:
- IC1 pad 42: (no net) -> Net-(IC1-Pad42)
Routing:
- net Net-(IC1-Pad42): track 0.00 -> 23.3 mm
- net Earth: track 286.0 -> 286.5 mm
Changed lines of the file:
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@@
-(kicad_pcb (version 4) (host pcbnew 4.0.2+dfsg1-stable)
+(kicad_pcb (version 4) (host pcbnew 4.0.5-e0-6337~49~ubuntu16.04.1)
   (general
-    (links 100)
+    (links 104)
     (no_connects 1)
-    (area -37.132143 -30.144049 31.932143 27.475)
+    (area -37.075001 -25.075001 25.075001 25.075001)
     (thickness 1.6)
     (drawings 25)
-    (tracks 470)
+    (tracks 481)
     (zones 0)
-    (modules 42)
-    (nets 42)
+    (modules 43)
+    (nets 43)
   )
   (page A4)
@@
   (net 40 "Net-(Q4-Pad3)")
   (net 41 "Net-(Q5-Pad3)")
+  (net 42 "Net-(IC1-Pad42)")
   (net_class Default "This is the default net class."
     (clearance 0.2)
@@
     (add_net "Net-(IC1-Pad21)")
     (add_net "Net-(IC1-Pad22)")
+    (add_net "Net-(IC1-Pad42)")
     (add_net "Net-(IC1-Pad43)")
     (add_net "Net-(IC1-Pad44)")
@@
     (pad 40 smd rect (at 1 7.7 90) (size 1.5 0.3) (layers F.Cu F.Paste F.Mask))
     (pad 41 smd rect (at 1.5 7.7 90) (size 1.5 0.3) (layers F.Cu F.Paste F.Mask))
-    (pad 42 smd rect (at 2 7.7 90) (size 1.5 0.3) (layers F.Cu F.Paste F.Mask))
+    (pad 42 smd rect (at 2 7.7 90) (size 1.5 0.3) (layers F.Cu F.Paste F.Mask)
+      (net 42 "Net-(IC1-Pad42)"))
     (pad 43 smd rect (at 2.5 7.7 90) (size 1.5 0.3) (layers F.Cu F.Paste F.Mask)
       (net 20 "Net-(IC1-Pad43)"))
@@
       (net 3 "Net-(C2-Pad1)"))
   )
+  (module Switches:PanasonicEVQPU_SPST_NO (layer F.Cu)
+    (at 7 25)
+    (fp_text reference SW1 (at 0 -5.5) (layer F.SilkS)
+      (effects (font (size 1 1) (thickness 0.15)))
+    )
+    (fp_text value SW_SPST (at 0 -7) (layer F.Fab)
+      (effects (font (size 1 1) (thickness 0.15)))
+    )
+    (fp_line (start 2.35 -0.8) (end 2.35 -0.5) (layer F.SilkS) (width 0.15))
+    (fp_line (start -2.35 -0.8) (end -2.35 -0.5) (layer F.SilkS) (width 0.15))
+    (fp_line (start 2.35 -4) (end 2.35 -3.7) (layer F.SilkS) (width 0.15))
+    (fp_line (start -2.35 -4) (end -2.35 -3.7) (layer F.SilkS) (width 0.15))
+    (fp_line (start 2.35 -2.5) (end 2.35 -2) (layer F.SilkS) (width 0.15))
+    (fp_line (start -2.35 -2.5) (end -2.35 -2) (layer F.SilkS) (width 0.15))
+    (fp_line (start 0.5 -4) (end 2.35 -4) (layer F.SilkS) (width 0.15))
+    (fp_line (start -2.35 -4) (end -0.5 -4) (layer F.SilkS) (width 0.15))
+    (pad "" np_thru_hole circle (at 0 -3.625) (size 0.75 0.75) (drill 0.75) (layers *.Cu *.Mask))
+    (pad 2 smd rect (at 2.625 -3.1) (size 1.55 1) (layers F.Cu F.Paste F.Mask)
+      (net 42 "Net-(IC1-Pad42)"))
+    (pad 2 smd rect (at -2.625 -3.1) (size 1.55 1) (layers F.Cu F.Paste F.Mask)
+      (net 42 "Net-(IC1-Pad42)"))
+    (pad 1 smd rect (at 2.625 -1.4) (size 1.55 1) (layers F.Cu F.Paste F.Mask)
+      (net 2 Earth))
+    (pad 1 smd rect (at -2.625 -1.4) (size 1.55 1) (layers F.Cu F.Paste F.Mask)
+      (net 2 Earth))
+    (pad "" np_thru_hole circle (at 0 -0.875) (size 0.75 0.75) (drill 0.75) (layers *.Cu *.Mask))
+  )
   (gr_text "University of Tokyo\nBL-Ctrl to PWM V2\nChris Raabe 2017" (at 17 16.999 45) (layer F.SilkS)
     (effects (font (size 1 1) (thickness 0.15)))
@@
   (segment (start -3.5 16.13) (end -3.6 16.13) (width 0.25) (layer F.Cu) (net 1))
   (segment (start -3.6 16.13) (end -6.25 16.13) (width 0.25) (layer F.Cu) (net 1))
+  (segment (start 0.206 22.206) (end 0.294 22.206) (width 0.25) (layer F.Cu) (net 2))
+  (segment (start 4.25 18.25) (end 4.25 16.13) (width 0.25) (layer F.Cu) (net 2))
+  (segment (start 0.294 22.206) (end 4.25 18.25) (width 0.25) (layer F.Cu) (net 2))
+  (segment (start -2.14 22.206) (end 0.206 22.206) (width 0.25) (layer F.Cu) (net 2))
+  (segment (start -2.14 22.206) (end -10.522 22.206) (width 0.25) (layer B.Cu) (net 2))
+  (segment (start -10.522 22.206) (end -11.03 21.698) (width 0.25) (layer B.Cu) (net 2))
+  (via (at -2.14 22.206) (size 0.6) (drill 0.4) (layers F.Cu B.Cu) (net 2))
+  (segment (start -8.77 16.11) (end -11.03 16.11) (width 0.25) (layer F.Cu) (net 2))
+  (via (at -11.03 16.11) (size 0.6) (drill 0.4) (layers F.Cu B.Cu) (net 2))
+  (segment (start -11.03 21.698) (end -11.03 16.11) (width 0.25) (layer B.Cu) (net 2))
+  (segment (start 1.6 23.6) (end 4.375 23.6) (width 0.25) (layer F.Cu) (net 2))
+  (segment (start 0.206 22.206) (end 1.6 23.6) (width 0.25) (layer F.Cu) (net 2))
   (segment (start 3.25 -11.75) (end 3.25 -16.75) (width 0.25) (layer B.Cu) (net 2))
   (via (at 3.25 -16.75) (size 0.6) (drill 0.4) (layers F.Cu B.Cu) (net 2))
@@
   (segment (start -4.979997 -6.160999) (end -4.679998 -5.861) (width 0.25) (layer F.Cu) (net 2))
   (via (at -4.679998 -5.861) (size 0.6) (drill 0.4) (layers F.Cu B.Cu) (net 2))
-  (segment (start -2.14 22.206) (end -10.522 22.206) (width 0.25) (layer B.Cu) (net 2))
-  (segment (start -10.522 22.206) (end -11.03 21.698) (width 0.25) (layer B.Cu) (net 2))
-  (segment (start -11.03 21.698) (end -11.03 16.11) (width 0.25) (layer B.Cu) (net 2))
   (segment (start -5.95 -0.4) (end -5.442 -0.4) (width 0.25) (layer F.Cu) (net 2))
   (segment (start -5.442 -0.4) (end -4.68 0.362) (width 0.25) (layer F.Cu) (net 2))
@@
   (segment (start 20.733 8.109) (end 19.069 8.109) (width 0.25) (layer B.Cu) (net 2))
   (segment (start 22.365 6.477) (end 20.733 8.109) (width 0.25) (layer B.Cu) (net 2))
-  (segment (start 6.496 16.11) (end 6.496 21.571) (width 0.25) (layer F.Cu) (net 2))
-  (segment (start 6.496 21.571) (end 5.861 22.206) (width 0.25) (layer F.Cu) (net 2))
-  (segment (start 5.861 22.206) (end -2.14 22.206) (width 0.25) (layer F.Cu) (net 2))
   (segment (start -7.7 -1) (end -8.7 -1) (width 0.25) (layer F.Cu) (net 2))
   (segment (start 7.766 7.728) (end 6.496 8.998) (width 0.25) (layer B.Cu) (net 2))
@@
   (segment (start -8.75 12.306) (end -8.75 16.13) (width 0.25) (layer F.Cu) (net 2))
   (segment (start -6.25 12.25) (end -8.694 12.25) (width 0.25) (layer F.Cu) (net 2))
-  (segment (start -11.03 16.11) (end -8.77 16.11) (width 0.25) (layer F.Cu) (net 2))
   (segment (start -8.77 16.11) (end -8.75 16.13) (width 0.25) (layer F.Cu) (net 2))
-  (via (at -11.03 16.11) (size 0.6) (drill 0.4) (layers F.Cu B.Cu) (net 2))
-  (via (at -2.14 22.206) (size 0.6) (drill 0.4) (layers F.Cu B.Cu) (net 2))
   (segment (start 6.496 16.11) (end 4.27 16.11) (width 0.25) (layer F.Cu) (net 2))
   (segment (start 4.27 16.11) (end 4.25 16.13) (width 0.25) (layer F.Cu) (net 2))
@@
   (segment (start -23 14) (end -21.5 12.5) (width 0.25) (layer F.Cu) (net 40))
   (segment (start -24.65 16) (end -20 16) (width 0.25) (layer F.Cu) (net 41))
+  (segment (start 4.375 21.9) (end 5.65 21.9) (width 0.25) (layer F.Cu) (net 42))
+  (segment (start 8.35 21.9) (end 9.625 21.9) (width 0.25) (layer F.Cu) (net 42))
+  (segment (start 7.5 22.75) (end 8.35 21.9) (width 0.25) (layer F.Cu) (net 42))
+  (segment (start 6.5 22.75) (end 7.5 22.75) (width 0.25) (layer F.Cu) (net 42))
+  (segment (start 5.65 21.9) (end 6.5 22.75) (width 0.25) (layer F.Cu) (net 42))
+  (segment (start 2 7.7) (end 2 8.75) (width 0.25) (layer F.Cu) (net 42))
+  (segment (start 9.625 16.375) (end 9.625 21.9) (width 0.25) (layer F.Cu) (net 42))
+  (segment (start 2 8.75) (end 9.625 16.375) (width 0.25) (layer F.Cu) (net 42))
   (zone (net 2) (net_name Earth) (layer F.Cu) (hatch edge 0.508)
     (connect_pads (clearance 0.508))
